File: schematics/4d7s_74hs595.sch (KiCad schematic (older format))
At the start: 12 parts, among them J1 C1, U1 74HC595, U2 YSD-439AY2B-35, U3 74HC595

Commit message: Conectado el pin para el punto en el display. Eliminados avisos por la alimentación.
Parts:
- added R8: 330, Resistor_THT:R_Axial_DIN0204_L3.6mm_D1.6mm_P1.90mm_Vertical, symbol Device:R
Connections:
- net labels removed: +5V
- wire segments 95 -> 102
- no-connect marks 11 -> 9
Other:
- moved on the sheet: C1, J1, R1, R2, R3, R4, R5, R6, R7, U1, U2, U3
